File: hardware/chipiplex_4_12_leds.kicad_sch (KiCad schematic)
At the start: 17 parts, among them Q1 MMBT3906, Q2 MMBT3906, Q3 MMBT3906, Q4 MMBT3906

Commit message: [Hardware] Replace LISDH Motion Sensor with LSM6DSM
Change motion sensor to an accelerometer + gyro unit. Route the second interrupt line to the STM32.
Parts:
- renumbered D5 to D29, D7 to D30, D9 to D31, D17 to D32, D18 to D33, D19 to D34, D11 to D35, D12 to D36, D13 to D37, Q2 to Q10, Q3 to Q11, Q4 to Q12, Q1 to Q9, R15 to R33, R16 to R34, R17 to R35, R18 to R36
Changed lines of the file:
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@@
 		(dnp no)
 		(fields_autoplaced yes)
-		(property "Reference" "D19"
+		(property "Reference" "D34"
 			(at 101.6 103.1874 90)
 			(effects
@@
 				(path "/addc3208-a9c4-4d28-9808-559c1d81e43b/0fdb39f4-f262-4df8-82d6-8f176468da30/00cf998d-e4a1-4a22-8ba8-d5d4d57b1c62"
 					(reference "D34")
-					(unit 1)
-				)
-				(path "/addc3208-a9c4-4d28-9808-559c1d81e43b/0fdb39f4-f262-4df8-82d6-8f176468da30/46bf3b19-1647-4409-ae4c-bb996d695482"
-					(reference "D19")
-					(unit 1)
-				)
-				(path "/addc3208-a9c4-4d28-9808-559c1d81e43b/0fdb39f4-f262-4df8-82d6-8f176468da30/a55ea924-f9da-4eb7-9a51-aee60932cddf"
-					(reference "D22")
 					(unit 1)
 				)
@@
 		(on_board yes)
 		(dnp no)
-		(property "Reference" "Q3"
+		(property "Reference" "Q11"
 			(at 156.21 57.1499 0)
 			(effects
@@
 					(unit 1)
 				)
-				(path "/addc3208-a9c4-4d28-9808-559c1d81e43b/0fdb39f4-f262-4df8-82d6-8f176468da30/46bf3b19-1647-4409-ae4c-bb996d695482"
-					(reference "Q3")
-					(unit 1)
-				)
-				(path "/addc3208-a9c4-4d28-9808-559c1d81e43b/0fdb39f4-f262-4df8-82d6-8f176468da30/a55ea924-f9da-4eb7-9a51-aee60932cddf"
-					(reference "Q7")
-					(unit 1)
-				)
 			)
 		)
@@
 		(dnp no)
 		(fields_autoplaced yes)
-		(property "Reference" "D5"
+		(property "Reference" "D29"
 			(at 50.8 75.2474 90)
 			(effects
@@
 					(unit 1)
 				)
-				(path "/addc3208-a9c4-4d28-9808-559c1d81e43b/0fdb39f4-f262-4df8-82d6-8f176468da30/46bf3b19-1647-4409-ae4c-bb996d695482"
-					(reference "D5")
-					(unit 1)
-				)
-				(path "/addc3208-a9c4-4d28-9808-559c1d81e43b/0fdb39f4-f262-4df8-82d6-8f176468da30/a55ea924-f9da-4eb7-9a51-aee60932cddf"
-					(reference "D6")
-					(unit 1)
-				)
 			)
 		)
@@
 		(dnp no)
 		(fields_autoplaced yes)
-		(property "Reference" "D18"
+		(property "Reference" "D33"
 			(at 101.6 89.2174 90)
 			(effects
@@
 					(unit 1)
 				)
-				(path "/addc3208-a9c4-4d28-9808-559c1d81e43b/0fdb39f4-f262-4df8-82d6-8f176468da30/46bf3b19-1647-4409-ae4c-bb996d695482"
-					(reference "D18")
-					(unit 1)
-				)
-				(path "/addc3208-a9c4-4d28-9808-559c1d81e43b/0fdb39f4-f262-4df8-82d6-8f176468da30/a55ea924-f9da-4eb7-9a51-aee60932cddf"
-					(reference "D21")
-					(unit 1)
-				)
 			)
 		)
@@
 		(on_board yes)
 		(dnp no)
-		(property "Reference" "R16"
+		(property "Reference" "R34"
 			(at 88.9 50.7999 0)
 			(effects
@@
 					(unit 1)
 				)
-				(path "/addc3208-a9c4-4d28-9808-559c1d81e43b/0fdb39f4-f262-4df8-82d6-8f176468da30/46bf3b19-1647-4409-ae4c-bb996d695482"
-					(reference "R16")
-					(unit 1)
-				)
-				(path "/addc3208-a9c4-4d28-9808-559c1d81e43b/0fdb39f4-f262-4df8-82d6-8f176468da30/a55ea924-f9da-4eb7-9a51-aee60932cddf"
-					(reference "R20")
-					(unit 1)
-				)
 			)
 		)
@@
 		(dnp no)
 		(fields_autoplaced yes)
-		(property "Reference" "D11"
+		(property "Reference" "D35"
 			(at 156.21 73.9774 90)
 			(effects
@@
 					(unit 1)
 				)
-				(path "/addc3208-a9c4-4d28-9808-559c1d81e43b/0fdb39f4-f262-4df8-82d6-8f176468da30/46bf3b19-1647-4409-ae4c-bb996d695482"
-					(reference "D11")
-					(unit 1)
-				)
-				(path "/addc3208-a9c4-4d28-9808-559c1d81e43b/0fdb39f4-f262-4df8-82d6-8f176468da30/a55ea924-f9da-4eb7-9a51-aee60932cddf"
-					(reference "D14")
-					(unit 1)
-				)
 			)
 		)
@@
 		(dnp no)
 		(fields_autoplaced yes)
-		(property "Reference" "D17"
+		(property "Reference" "D32"
 			(at 101.6 75.2474 90)
 			(effects
@@
 					(unit 1)
 				)
-				(path "/addc3208-a9c4-4d28-9808-559c1d81e43b/0fdb39f4-f262-4df8-82d6-8f176468da30/46bf3b19-1647-4409-ae4c-bb996d695482"
-					(reference "D17")
-					(unit 1)
-				)
-				(path "/addc3208-a9c4-4d28-9808-559c1d81e43b/0fdb39f4-f262-4df8-82d6-8f176468da30/a55ea924-f9da-4eb7-9a51-aee60932cddf"
-					(reference "D20")
-					(unit 1)
-				)
 			)
 		)
@@
 		(on_board yes)
 		(dnp no)
-		(property "Reference" "R17"
+		(property "Reference" "R35"
 			(at 143.51 50.7999 0)
 			(effects
@@
 					(unit 1)
 				)
-				(path "/addc3208-a9c4-4d28-9808-559c1d81e43b/0fdb39f4-f262-4df8-82d6-8f176468da30/46bf3b19-1647-4409-ae4c-bb996d695482"
-					(reference "R17")
-					(unit 1)
-				)
-				(path "/addc3208-a9c4-4d28-9808-559c1d81e43b/0fdb39f4-f262-4df8-82d6-8f176468da30/a55ea924-f9da-4eb7-9a51-aee60932cddf"
-					(reference "R21")
-					(unit 1)
-				)
 			)
 		)
@@
 		(on_board yes)
 		(dnp no)
-		(property "Reference" "D9"
+		(property "Reference" "D31"
 			(at 50.8 103.1874 90)
 			(effects
@@
 				(path "/addc3208-a9c4-4d28-9808-559c1d81e43b/0fdb39f4-f262-4df8-82d6-8f176468da30/00cf998d-e4a1-4a22-8ba8-d5d4d57b1c62"
 					(reference "D31")
-					(unit 1)
-				)
-				(path "/addc3208-a9c4-4d28-9808-559c1d81e43b/0fdb39f4-f262-4df8-82d6-8f176468da30/46bf3b19-1647-4409-ae4c-bb996d695482"
-					(reference "D9")
-					(unit 1)
-				)
-				(path "/addc3208-a9c4-4d28-9808-559c1d81e43b/0fdb39f4-f262-4df8-82d6-8f176468da30/a55ea924-f9da-4eb7-9a51-aee60932cddf"
-					(reference "D10")
 					(unit 1)
 				)
@@
 		(on_board yes)
 		(dnp no)
-		(property "Reference" "Q2"
+		(property "Reference" "Q10"
 			(at 101.6 57.1499 0)
 			(effects
@@
 					(unit 1)
 				)
-				(path "/addc3208-a9c4-4d28-9808-559c1d81e43b/0fdb39f4-f262-4df8-82d6-8f176468da30/46bf3b19-1647-4409-ae4c-bb996d695482"
-					(reference "Q2")
-					(unit 1)
-				)
-				(path "/addc3208-a9c4-4d28-9808-559c1d81e43b/0fdb39f4-f262-4df8-82d6-8f176468da30/a55ea924-f9da-4eb7-9a51-aee60932cddf"
-					(reference "Q6")
-					(unit 1)
-				)
 			)
 		)
@@
 		(dnp no)
 		(fields_autoplaced yes)
-		(property "Reference" "D13"
+		(property "Reference" "D37"
 			(at 156.21 101.9174 90)
 			(effects
@@
 					(unit 1)
 				)
-				(path "/addc3208-a9c4-4d28-9808-559c1d81e43b/0fdb39f4-f262-4df8-82d6-8f176468da30/46bf3b19-1647-4409-ae4c-bb996d695482"
-					(reference "D13")
-					(unit 1)
-				)
-				(path "/addc3208-a9c4-4d28-9808-559c1d81e43b/0fdb39f4-f262-4df8-82d6-8f176468da30/a55ea924-f9da-4eb7-9a51-aee60932cddf"
-					(reference "D16")
-					(unit 1)
-				)
 			)
 		)
@@
 		(dnp no)
 		(fields_autoplaced yes)
-		(property "Reference" "D7"
+		(property "Reference" "D30"
 			(at 50.8 89.2174 90)
 			(effects
@@
 					(unit 1)
 				)
-				(path "/addc3208-a9c4-4d28-9808-559c1d81e43b/0fdb39f4-f262-4df8-82d6-8f176468da30/46bf3b19-1647-4409-ae4c-bb996d695482"
-					(reference "D7")
-					(unit 1)
-				)
-				(path "/addc3208-a9c4-4d28-9808-559c1d81e43b/0fdb39f4-f262-4df8-82d6-8f176468da30/a55ea924-f9da-4eb7-9a51-aee60932cddf"
-					(reference "D8")
-					(unit 1)
-				)
 			)
 		)
@@
 		(dnp no)
 		(fields_autoplaced yes)
-		(property "Reference" "D12"
+		(property "Reference" "D36"
 			(at 156.21 87.9474 90)
 			(effects
@@
 					(unit 1)
 				)
-				(path "/addc3208-a9c4-4d28-9808-559c1d81e43b/0fdb39f4-f262-4df8-82d6-8f176468da30/46bf3b19-1647-4409-ae4c-bb996d695482"
-					(reference "D12")
-					(unit 1)
-				)
-				(path "/addc3208-a9c4-4d28-9808-559c1d81e43b/0fdb39f4-f262-4df8-82d6-8f176468da30/a55ea924-f9da-4eb7-9a51-aee60932cddf"
-					(reference "D15")
-					(unit 1)
-				)
 			)
 		)
@@
 		(on_board yes)
 		(dnp no)
-		(property "Reference" "R18"
+		(property "Reference" "R36"
 			(at 194.31 50.7999 0)
 			(effects
@@
 				(path "/addc3208-a9c4-4d28-9808-559c1d81e43b/0fdb39f4-f262-4df8-82d6-8f176468da30/00cf998d-e4a1-4a22-8ba8-d5d4d57b1c62"
 					(reference "R36")
-					(unit 1)
-				)
-				(path "/addc3208-a9c4-4d28-9808-559c1d81e43b/0fdb39f4-f262-4df8-82d6-8f176468da30/46bf3b19-1647-4409-ae4c-bb996d695482"
-					(reference "R18")
-					(unit 1)
-				)
-				(path "/addc3208-a9c4-4d28-9808-559c1d81e43b/0fdb39f4-f262-4df8-82d6-8f176468da30/a55ea924-f9da-4eb7-9a51-aee60932cddf"
-					(reference "R22")
 					(unit 1)
 				)
@@
 		(on_board yes)
 		(dnp no)
-		(property "Reference" "Q1"
+		(property "Reference" "Q9"
 			(at 50.8 57.1499 0)
 			(effects
@@
 				(path "/addc3208-a9c4-4d28-9808-559c1d81e43b/0fdb39f4-f262-4df8-82d6-8f176468da30/00cf998d-e4a1-4a22-8ba8-d5d4d57b1c62"
 					(reference "Q9")
-					(unit 1)
-				)
-				(path "/addc3208-a9c4-4d28-9808-559c1d81e43b/0fdb39f4-f262-4df8-82d6-8f176468da30/46bf3b19-1647-4409-ae4c-bb996d695482"
-					(reference "Q1")
-					(unit 1)
-				)
-				(path "/addc3208-a9c4-4d28-9808-559c1d81e43b/0fdb39f4-f262-4df8-82d6-8f176468da30/a55ea924-f9da-4eb7-9a51-aee60932cddf"
-					(reference "Q5")
 					(unit 1)
 				)
@@
 		(on_board yes)
 		(dnp no)
-		(property "Reference" "Q4"
+		(property "Reference" "Q12"
 			(at 207.01 57.1499 0)
 			(effects
@@
 					(unit 1)
 				)
-				(path "/addc3208-a9c4-4d28-9808-559c1d81e43b/0fdb39f4-f262-4df8-82d6-8f176468da30/46bf3b19-1647-4409-ae4c-bb996d695482"
-					(reference "Q4")
-					(unit 1)
-				)
-				(path "/addc3208-a9c4-4d28-9808-559c1d81e43b/0fdb39f4-f262-4df8-82d6-8f176468da30/a55ea924-f9da-4eb7-9a51-aee60932cddf"
-					(reference "Q8")
-					(unit 1)
-				)
 			)
 		)
@@
 		(on_board yes)
 		(dnp no)
-		(property "Reference" "R15"
+		(property "Reference" "R33"
 			(at 38.1 50.7999 0)
 			(effects
@@
 					(unit 1)
 				)
-				(path "/addc3208-a9c4-4d28-9808-559c1d81e43b/0fdb39f4-f262-4df8-82d6-8f176468da30/46bf3b19-1647-4409-ae4c-bb996d695482"
-					(reference "R15")
-					(unit 1)
-				)
-				(path "/addc3208-a9c4-4d28-9808-559c1d81e43b/0fdb39f4-f262-4df8-82d6-8f176468da30/a55ea924-f9da-4eb7-9a51-aee60932cddf"
-					(reference "R19")
-					(unit 1)
-				)

Commit message: Change many passives to 0402 and assign part numbers
Incorporate 0402 parts where possible
Assign Manufacturer Part Numbers to parts where possible
Update layout for the new passive sizes
Parts:
- D29, D30, D31, D32, D33, D34, D35, D36, D37: MPN (none) -> LTST-C171GKT
- Q10, Q11, Q12, Q9: MPN (none) -> MMBT3906
- R33, R34, R35, R36: footprint Resistor_SMD:R_0603_1608Metric_Pad0.98x0.95mm_HandSolder -> Resistor_SMD:R_0402_1005Metric; MPN (none) -> RC0402JR-0750RL
Changed lines of the file:
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@@
+			)
+		)
+		(property "MPN" "LTST-C171GKT"
+			(at 97.79 102.87 0)
+			(effects
+				(font
+					(size 1.27 1.27)
+				)
+				(hide yes)
 			)
 		)
@@
 			)
 		)
+		(property "MPN" "MMBT3906"
+			(at 151.13 58.42 0)
+			(effects
+				(font
+					(size 1.27 1.27)
+				)
+				(hide yes)
+			)
+		)
 		(pin "1"
 		)
@@
 			)
 		)
+		(property "MPN" "LTST-C171GKT"
+			(at 46.99 74.93 0)
+			(effects
+				(font
+					(size 1.27 1.27)
+				)
+				(hide yes)
+			)
+		)
 		(pin "1"
 		)
@@
 			)
 		)
+		(property "MPN" "LTST-C171GKT"
+			(at 97.79 88.9 0)
+			(effects
+				(font
+					(size 1.27 1.27)
+				)
+				(hide yes)
+			)
+		)
 		(pin "1"
 		)
@@
 			)
 		)
-		(property "Footprint" "Resistor_SMD:R_0603_1608Metric_Pad0.98x0.95mm_HandSolder"
+		(property "Footprint" "Resistor_SMD:R_0402_1005Metric"
 			(at 89.662 52.07 90)
 			(effects
@@
 		)
 		(property "Description" "Resistor"
+			(at 91.44 52.07 0)
+			(effects
+				(font
+					(size 1.27 1.27)
+				)
+				(hide yes)
+			)
+		)
+		(property "MPN" "RC0402JR-0750RL"
 			(at 91.44 52.07 0)
 			(effects
@@
 			)
 		)
+		(property "MPN" "LTST-C171GKT"
+			(at 152.4 73.66 0)
+			(effects
+				(font
+					(size 1.27 1.27)
+				)
+				(hide yes)
+			)
+		)
 		(pin "1"
 		)
@@
 			)
 		)
+		(property "MPN" "LTST-C171GKT"
+			(at 97.79 74.93 0)
+			(effects
+				(font
+					(size 1.27 1.27)
+				)
+				(hide yes)
+			)
+		)
 		(pin "1"
 		)
@@
 			)
 		)
-		(property "Footprint" "Resistor_SMD:R_0603_1608Metric_Pad0.98x0.95mm_HandSolder"
+		(property "Footprint" "Resistor_SMD:R_0402_1005Metric"
 			(at 144.272 52.07 90)
 			(effects
@@
 			)
 		)
+		(property "MPN" "RC0402JR-0750RL"
+			(at 146.05 52.07 0)
+			(effects
+				(font
+					(size 1.27 1.27)
+				)
+				(hide yes)
+			)
+		)
 		(pin "1"
 		)
@@
 		)
 		(property "Description" "Light emitting diode"
+			(at 46.99 102.87 0)
+			(effects
+				(font
+					(size 1.27 1.27)
+				)
+				(hide yes)
+			)
+		)
+		(property "MPN" "LTST-C171GKT"
 			(at 46.99 102.87 0)
 			(effects
@@
 			)
 		)
+		(property "MPN" "MMBT3906"
+			(at 96.52 58.42 0)
+			(effects
+				(font
+					(size 1.27 1.27)
+				)
+				(hide yes)
+			)
+		)
 		(pin "1"
 		)
@@
 			)
 		)
+		(property "MPN" "LTST-C171GKT"
+			(at 152.4 101.6 0)
+			(effects
+				(font
+					(size 1.27 1.27)
+				)
+				(hide yes)
+			)
+		)
 		(pin "1"
 		)
@@
 			)
 		)
+		(property "MPN" "LTST-C171GKT"
+			(at 46.99 88.9 0)
+			(effects
+				(font
+					(size 1.27 1.27)
+				)
+				(hide yes)
+			)
+		)
 		(pin "1"
 		)
@@
 			)
 		)
+		(property "MPN" "LTST-C171GKT"
+			(at 152.4 87.63 0)
+			(effects
+				(font
+					(size 1.27 1.27)
+				)
+				(hide yes)
+			)
+		)
 		(pin "1"
 		)
@@
 			)
 		)
-		(property "Footprint" "Resistor_SMD:R_0603_1608Metric_Pad0.98x0.95mm_HandSolder"
+		(property "Footprint" "Resistor_SMD:R_0402_1005Metric"
 			(at 195.072 52.07 90)
 			(effects
@@
 		)
 		(property "Description" "Resistor"
+			(at 196.85 52.07 0)
+			(effects
+				(font
+					(size 1.27 1.27)
+				)
+				(hide yes)
+			)
+		)
+		(property "MPN" "RC0402JR-0750RL"
 			(at 196.85 52.07 0)
 			(effects
@@
 			)
 		)
+		(property "MPN" "MMBT3906"
+			(at 45.72 58.42 0)
+			(effects
+				(font
+					(size 1.27 1.27)
+				)
+				(hide yes)
+			)
+		)
 		(pin "1"
 		)
@@
 			)
 		)
+		(property "MPN" "MMBT3906"
+			(at 201.93 58.42 0)
+			(effects
+				(font
+					(size 1.27 1.27)
+				)
+				(hide yes)
+			)
+		)
 		(pin "1"
 		)
@@
 			)
 		)
-		(property "Footprint" "Resistor_SMD:R_0603_1608Metric_Pad0.98x0.95mm_HandSolder"
+		(property "Footprint" "Resistor_SMD:R_0402_1005Metric"
 			(at 38.862 52.07 90)
 			(effects
@@
 			(at 40.64 52.07 0)
 			(effects
+				(font
+					(size 1.27 1.27)
+				)
+				(hide yes)
+			)
+		)
+		(property "MPN" "RC0402JR-0750RL"
+			(at 40.64 52.07 0)
+			(effects
