File: hardware/power.kicad_sch (KiCad schematic)
At the start: 9 parts, among them U2 TPS61200DRC

Commit message: [Hardware] Boost converter updates.
* Tie PS (power save) pin to ground to enable higher efficiencies during low-current operation
* Add 0ohm resistor at output pin to measure current.
Parts:
- added R13, R14: 0, Resistor_SMD:R_0603_1608Metric_Pad0.98x0.95mm_HandSolder, symbol Device:R
Connections:
- net 3V3: now also R14.2; no longer C11.1, R4.1, U2.2 (VOUT)
- net GND: now also R13.2
- net at C23.1, C9.1, JP2.2 (C)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: no longer U2.8 (PS)
- new net: C11.1, R14.1, R4.1, U2.2 (VOUT)
- new net: R13.1, U2.8 (PS)

Commit message: Change many passives to 0402 and assign part numbers
Incorporate 0402 parts where possible
Assign Manufacturer Part Numbers to parts where possible
Update layout for the new passive sizes
Parts:
- C10: footprint Capacitor_SMD:C_0603_1608Metric_Pad1.08x0.95mm_HandSolder -> Capacitor_SMD:C_0402_1005Metric; MPN (none) -> CL05A104KA5NNNC
- C11, C23: MPN (none) -> CL10A106MQ8NNNC
- C9: footprint Capacitor_SMD:C_0603_1608Metric_Pad1.08x0.95mm_HandSolder -> Capacitor_SMD:C_0402_1005Metric; MPN (none) -> CL05A475MP5NRNC
- L1: MPN (none) -> LPS3015-222MRC
- R13, R14: footprint Resistor_SMD:R_0603_1608Metric_Pad0.98x0.95mm_HandSolder -> Resistor_SMD:R_0402_1005Metric; MPN (none) -> RC0402JR-070RL
- R4: footprint Resistor_SMD:R_0603_1608Metric_Pad0.98x0.95mm_HandSolder -> Resistor_SMD:R_0402_1005Metric; MPN (none) -> RC0402FR-071ML
- R5: footprint Resistor_SMD:R_0603_1608Metric_Pad0.98x0.95mm_HandSolder -> Resistor_SMD:R_0402_1005Metric; MPN (none) -> RC0402JR-07180KL
- U2: MPN (none) -> TPS61200DRCT
Changed lines of the file:
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@@
+			)
+		)
+		(property "MPN" "CL10A106MQ8NNNC"
+			(at 232.41 96.52 0)
+			(effects
+				(font
+					(size 1.27 1.27)
+				)
+				(hide yes)
 			)
 		)
@@
 			)
 		)
+		(property "MPN" "TPS61200DRCT"
+			(at 195.58 95.25 0)
+			(effects
+				(font
+					(size 1.27 1.27)
+				)
+				(hide yes)
+			)
+		)
 		(pin "3"
 		)
@@
 			)
 		)
+		(property "MPN" ""
+			(at 161.29 78.74 0)
+			(effects
+				(font
+					(size 1.27 1.27)
+				)
+				(hide yes)
+			)
+		)
 		(pin "2"
 		)
@@
 			)
 		)
-		(property "Footprint" "Resistor_SMD:R_0603_1608Metric_Pad0.98x0.95mm_HandSolder"
+		(property "Footprint" "Resistor_SMD:R_0402_1005Metric"
 			(at 219.202 96.52 90)
 			(effects
@@
 		)
 		(property "Description" "Resistor"
+			(at 220.98 96.52 0)
+			(effects
+				(font
+					(size 1.27 1.27)
+				)
+				(hide yes)
+			)
+		)
+		(property "MPN" "RC0402FR-071ML"
 			(at 220.98 96.52 0)
 			(effects
@@
 			)
 		)
-		(property "Footprint" "Resistor_SMD:R_0603_1608Metric_Pad0.98x0.95mm_HandSolder"
+		(property "Footprint" "Resistor_SMD:R_0402_1005Metric"
 			(at 177.292 102.87 90)
 			(effects
@@
 		)
 		(property "Description" "Resistor"
+			(at 179.07 102.87 0)
+			(effects
+				(font
+					(size 1.27 1.27)
+				)
+				(hide yes)
+			)
+		)
+		(property "MPN" "RC0402JR-070RL"
 			(at 179.07 102.87 0)
 			(effects
@@
 			)
 		)
+		(property "MPN" "LPS3015-222MRC"
+			(at 195.58 77.47 0)
+			(effects
+				(font
+					(size 1.27 1.27)
+				)
+				(hide yes)
+			)
+		)
 		(pin "2"
 		)
@@
 			)
 		)
-		(property "Footprint" "Resistor_SMD:R_0603_1608Metric_Pad0.98x0.95mm_HandSolder"
+		(property "Footprint" "Resistor_SMD:R_0402_1005Metric"
 			(at 219.202 104.14 90)
 			(effects
@@
 		)
 		(property "Description" "Resistor"
+			(at 220.98 104.14 0)
+			(effects
+				(font
+					(size 1.27 1.27)
+				)
+				(hide yes)
+			)
+		)
+		(property "MPN" "RC0402JR-07180KL"
 			(at 220.98 104.14 0)
 			(effects
@@
 			)
 		)
-		(property "Footprint" "Resistor_SMD:R_0603_1608Metric_Pad0.98x0.95mm_HandSolder"
+		(property "Footprint" "Resistor_SMD:R_0402_1005Metric"
 			(at 232.41 90.678 90)
 			(effects
@@
 			)
 		)
+		(property "MPN" "RC0402JR-070RL"
+			(at 232.41 88.9 0)
+			(effects
+				(font
+					(size 1.27 1.27)
+				)
+				(hide yes)
+			)
+		)
 		(pin "2"
 		)
@@
 			)
 		)
+		(property "MPN" "CL10A106MQ8NNNC"
+			(at 161.29 95.25 0)
+			(effects
+				(font
+					(size 1.27 1.27)
+				)
+				(hide yes)
+			)
+		)
 		(pin "1"
 		)
@@
 			)
 		)
-		(property "Footprint" "Capacitor_SMD:C_0603_1608Metric_Pad1.08x0.95mm_HandSolder"
+		(property "Footprint" "Capacitor_SMD:C_0402_1005Metric"
 			(at 178.7652 119.38 0)
 			(effects
@@
 			)
 		)
+		(property "MPN" "CL05A104KA5NNNC"
+			(at 177.8 115.57 0)
+			(effects
+				(font
+					(size 1.27 1.27)
+				)
+				(hide yes)
+			)
+		)
 		(pin "1"
 		)
@@
 			)
 		)
-		(property "Footprint" "Capacitor_SMD:C_0603_1608Metric_Pad1.08x0.95mm_HandSolder"
+		(property "Footprint" "Capacitor_SMD:C_0402_1005Metric"
 			(at 176.2252 97.79 0)
 			(effects
@@
 			(at 175.26 93.98 0)
 			(effects
+				(font
+					(size 1.27 1.27)
+				)
+				(hide yes)
+			)
+		)
+		(property "MPN" "CL05A475MP5NRNC"
+			(at 175.26 93.98 0)
+			(effects

Commit message: Remove external power connector
Parts:
- removed JP2: Jumper_3_Bridged12, Jumper:SolderJumper-3_P1.3mm_Bridged2Bar12_Pad1.0x1.5mm_NumberLabels, symbol Jumper:Jumper_3_Bridged12
Connections:
- net VDC_BAT: now also C23.1, C9.1, L1.1, U2.5 (VIN), U2.6 (EN)
